File: PCB/Groove Coaster.kicad_pcb (KiCad board)
At the start: 2 copper layers, 28 parts

Commit message: All da changes
Parts:
- removed Joy1: JoyLeft_UP, Connector_JST:JST_XH_B2B-XH-A_1x02_P2.50mm_Vertical
- removed Joy2: JoyLeft_DOWN, Connector_JST:JST_XH_B2B-XH-A_1x02_P2.50mm_Vertical
- removed Joy3: JoyLeft_LEFT, Connector_JST:JST_XH_B2B-XH-A_1x02_P2.50mm_Vertical
- removed Joy4: JoyLeft_RIGHT, Connector_JST:JST_XH_B2B-XH-A_1x02_P2.50mm_Vertical
- removed Joy5: JoyRight_UP, Connector_JST:JST_XH_B2B-XH-A_1x02_P2.50mm_Vertical
- removed Joy6: JoyRight_DOWN, Connector_JST:JST_XH_B2B-XH-A_1x02_P2.50mm_Vertical
- removed Joy7: JoyRight_LEFT, Connector_JST:JST_XH_B2B-XH-A_1x02_P2.50mm_Vertical
- removed Joy8: JoyRight_RIGHT, Connector_JST:JST_XH_B2B-XH-A_1x02_P2.50mm_Vertical
- removed R10, R11, R6, R7, R8, R9: 10kΩ, Resistor_SMD:R_1206_3216Metric
- added J1: Conn_01x05, Connector_JST:JST_XH_B5B-XH-AM_1x05_P2.50mm_Vertical, F.Cu at (81.0, 75.0)
- added J2: Conn_01x05, Connector_JST:JST_XH_B5B-XH-AM_1x05_P2.50mm_Vertical, F.Cu at (98.1, 75.1)
- added REF**: MountingHole_3.2mm_M3_Pad, MountingHole:MountingHole_3.2mm_M3_Pad, F.Cu at (73.8, 80.9)
- added REF**: MountingHole_3.2mm_M3_Pad, MountingHole:MountingHole_3.2mm_M3_Pad, F.Cu at (73.6, 46.3)
- added REF**: MountingHole_3.2mm_M3_Pad, MountingHole:MountingHole_3.2mm_M3_Pad, F.Cu at (132.7, 46.3)
- added REF**: MountingHole_3.2mm_M3_Pad, MountingHole:MountingHole_3.2mm_M3_Pad, F.Cu at (132.8, 80.9)
- added U1: ProMicro, promicro:ProMicro-EnforcedTop, F.Cu at (93.3, 61.7)
- moved LED3 107.7 mm to (114.8, 48.9)
- moved LED1 95.8 mm to (130.4, 62.6)
- moved LED2 80.3 mm to (116.4, 76.3)
- moved BT1 75.2 mm to (83.4, 46.7)
- moved R12 72.4 mm to (116.6, 55.4), turned to 90 degrees
- moved R13 70.1 mm to (116.6, 60.5), turned to 90 degrees
- moved R14 69.6 mm to (116.6, 65.9), turned to 90 degrees
- moved R5 61.9 mm to (111.6, 60.5), turned to 90 degrees
- moved BT2 59.8 mm to (93.5, 46.9)
- moved R4 52.5 mm to (111.8, 65.9), turned to 90 degrees
- moved BT3 44.9 mm to (103.1, 46.8)
- moved R1 41.9 mm to (111.7, 55.2)
- moved R2 39.0 mm to (121.9, 57.8)
- moved R3 33.7 mm to (121.9, 63.7)
Routing:
- net Net-(R1-Pad2): track 0.00 -> 64.9 mm
- net Net-(LED3-+): track 0.00 -> 43.0 mm
- net Net-(LED1--): track 0.00 -> 36.8 mm
- net Net-(BT2-Pad2): track 0.00 -> 34.8 mm
- net Net-(LED3--): track 0.00 -> 32.4 mm
- net Net-(LED2--): track 0.00 -> 31.3 mm
- net Net-(BT3-Pad2): track 0.00 -> 28.9 mm
- net Net-(BT1-Pad2): track 0.00 -> 28.7 mm
- net Net-(U1-B2): track 0.00 -> 24.4 mm
- net Net-(J1-Pin_5): track 0.00 -> 24.0 mm
- net Net-(LED1-+): track 0.00 -> 19.4 mm
- net Net-(J2-Pin_5): track 0.00 -> 16.4 mm
- net Net-(J2-Pin_1): track 0.00 -> 16.4 mm
- net Net-(U1-B3): track 0.00 -> 14.1 mm
- net Net-(J1-Pin_3): track 0.00 -> 13.8 mm
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Other:
- board outline added: 69.8 x 45.3 mm
- net class Default removed
- board text added: "2023 BoredFish boredfish.dev"
- board text added: "GrooveTroller"
- board text added: "LETS GROOOOVE COASTER!"
- board text added: "Original by Anthony Raudino madewithhearts.com.au"

Commit message: oopies
Parts:
- removed LED1: BT1_LED, Connector_JST:JST_XH_B2B-XH-A_1x02_P2.50mm_Vertical
- removed LED2: BT2_LED, Connector_JST:JST_XH_B2B-XH-A_1x02_P2.50mm_Vertical
- removed LED3: BT3_LED, Connector_JST:JST_XH_B2B-XH-A_1x02_P2.50mm_Vertical
- removed the REF** at (73.8, 80.9)
- removed the REF** at (73.6, 46.3)
- removed the REF** at (132.7, 46.3)
- removed the REF** at (132.8, 80.9)
- added LEDGND1: Conn_01x03, Connector_JST:JST_XH_B3B-XH-A_1x03_P2.50mm_Vertical, F.Cu at (111.5, 46.1)
- added REF**: MountingHole_3.2mm_M3_ISO14580_Pad, MountingHole:MountingHole_3.2mm_M3_ISO14580_Pad, F.Cu at (125.6, 45.9)
- added REF**: MountingHole_3.2mm_M3_ISO14580_Pad, MountingHole:MountingHole_3.2mm_M3_ISO14580_Pad, F.Cu at (73.3, 81.2)
- added REF**: MountingHole_3.2mm_M3_ISO14580_Pad, MountingHole:MountingHole_3.2mm_M3_ISO14580_Pad, F.Cu at (125.6, 81.2)
- added REF**: MountingHole_3.2mm_M3_ISO14580_Pad, MountingHole:MountingHole_3.2mm_M3_ISO14580_Pad, F.Cu at (73.3, 45.9)
- BT1: value BT1_LeftJoyBtn -> Conn_01x02
- BT2: value BT2_RightJoyBtn -> Conn_01x02
- BT3: value BT3_StartBtn -> Conn_01x02
- moved BT3 1.88 mm to (101.4, 46.0)
- moved BT2 1.48 mm to (92.3, 46.0)
- moved BT1 0.81 mm to (83.0, 46.0)
Connections:
- U1 pad 17: Net-(LED1--) -> unconnected-(U1-F7-Pad17)
- U1 pad 18: Net-(LED2--) -> unconnected-(U1-F6-Pad18)
- U1 pad 19: Net-(LED3--) -> unconnected-(U1-F5-Pad19)
Routing:
- net Net-(LED1--): track 36.8 -> 0.00 mm
- net Net-(LED3--): track 32.4 -> 0.00 mm
- net Net-(LED2--): track 31.3 -> 0.00 mm
- net Net-(LEDGND1-Pin_2): track 12.8 -> 26.0 mm
- net Net-(LEDGND1-Pin_3): track 43.0 -> 31.3 mm
- net Net-(R1-Pad2): track 64.9 -> 71.8 mm
- net Net-(LEDGND1-Pin_1): track 19.4 -> 12.8 mm
- net Net-(BT3-Pin_1): track 8.71 -> 13.9 mm
- net Net-(J1-Pin_5): track 24.0 -> 28.6 mm
- net Net-(BT3-Pin_2): track 28.9 -> 33.4 mm
- net Net-(J2-Pin_4): track 10.8 -> 7.19 mm
- net Net-(J2-Pin_3): track 11.4 -> 7.90 mm
- net Net-(J2-Pin_1): track 16.4 -> 13.0 mm
- net Net-(BT2-Pin_2): track 34.8 -> 32.5 mm
- net Net-(BT1-Pin_2): track 28.7 -> 30.5 mm
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Other:
- board size 69.8 x 45.3 mm -> 62.3 x 45.3 mm

Commit message: pcbdeeznutz
Parts:
- J1, J2: footprint Connector_JST:JST_XH_B5B-XH-AM_1x05_P2.50mm_Vertical -> Connector_JST:JST_XH_B5B-XH-A_1x05_P2.50mm_Vertical
Changed lines of the file:
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@@
     )
   )
-  (footprint "Connector_JST:JST_XH_B5B-XH-AM_1x05_P2.50mm_Vertical" (layer "F.Cu")
+  (footprint "Connector_JST:JST_XH_B5B-XH-A_1x05_P2.50mm_Vertical" (layer "F.Cu")
     (at 81 75)
-    (descr "JST XH series connector, B5B-XH-AM, with boss (http://www.jst-mfg.com/product/pdf/eng/eXH.pdf), generated with kicad-footprint-generator")
-    (tags "connector JST XH vertical boss")
+    (descr "JST XH series connector, B5B-XH-A (http://www.jst-mfg.com/product/pdf/eng/eXH.pdf), generated with kicad-footprint-generator")
+    (tags "connector JST XH vertical")
     (property "Sheetfile" "Groove Coaster.kicad_sch")
     (property "Sheetname" "")
@@
     (fp_line (start -2.55 -0.2) (end -1.8 -0.2)
       (stroke (width 0.12) (type solid)) (layer "F.SilkS"))
-    (fp_line (start -1.8 -0.2) (end -1.8 1.14)
+    (fp_line (start -1.8 -0.2) (end -1.8 2.75)
+      (stroke (width 0.12) (type solid)) (layer "F.SilkS"))
+    (fp_line (start -1.8 2.75) (end 5 2.75)
       (stroke (width 0.12) (type solid)) (layer "F.SilkS"))
     (fp_line (start -1.6 -2.75) (end -2.85 -2.75)
@@
     (fp_line (start 0.75 -1.7) (end 9.25 -1.7)
       (stroke (width 0.12) (type solid)) (layer "F.SilkS"))
-    (fp_line (start 5 2.75) (end -0.74 2.75)
-      (stroke (width 0.12) (type solid)) (layer "F.SilkS"))
     (fp_line (start 9.25 -2.45) (end 0.75 -2.45)
       (stroke (width 0.12) (type solid)) (layer "F.SilkS"))
@@
     (fp_line (start 12.45 3.4) (end 12.45 -2.35)
       (stroke (width 0.1) (type solid)) (layer "F.Fab"))
-    (pad "" np_thru_hole circle (at -1.6 2) (size 1.2 1.2) (drill 1.2) (layers "*.Cu" "*.Mask"))
-    (pad "1" thru_hole roundrect (at 0 0) (size 1.7 1.95) (drill 0.95) (layers "*.Cu" "*.Mask") (roundrect_rratio 0.1470588235)
+    (pad "1" thru_hole roundrect (at 0 0) (size 1.7 1.95) (drill 0.95) (layers "*.Cu" "*.Mask") (roundrect_rratio 0.147059)
       (net 11 "Net-(J1-Pin_1)") (pinfunction "Pin_1") (pintype "passive"))
     (pad "2" thru_hole oval (at 2.5 0) (size 1.7 1.95) (drill 0.95) (layers "*.Cu" "*.Mask")
@@
     (pad "5" thru_hole oval (at 10 0) (size 1.7 1.95) (drill 0.95) (layers "*.Cu" "*.Mask")
       (net 15 "Net-(J1-Pin_5)") (pinfunction "Pin_5") (pintype "passive"))
-    (model "${KICAD6_3DMODEL_DIR}/Connector_JST.3dshapes/JST_XH_B5B-XH-AM_1x05_P2.50mm_Vertical.wrl"
+    (model "${KICAD6_3DMODEL_DIR}/Connector_JST.3dshapes/JST_XH_B5B-XH-A_1x05_P2.50mm_Vertical.wrl"
       (offset (xyz 0 0 0))
       (scale (xyz 1 1 1))
@@
     )
   )
-  (footprint "Connector_JST:JST_XH_B5B-XH-AM_1x05_P2.50mm_Vertical" (layer "F.Cu")
+  (footprint "Connector_JST:JST_XH_B5B-XH-A_1x05_P2.50mm_Vertical" (layer "F.Cu")
     (at 98.1 75.1)
-    (descr "JST XH series connector, B5B-XH-AM, with boss (http://www.jst-mfg.com/product/pdf/eng/eXH.pdf), generated with kicad-footprint-generator")
-    (tags "connector JST XH vertical boss")
+    (descr "JST XH series connector, B5B-XH-A (http://www.jst-mfg.com/product/pdf/eng/eXH.pdf), generated with kicad-footprint-generator")
+    (tags "connector JST XH vertical")
     (property "Sheetfile" "Groove Coaster.kicad_sch")
     (property "Sheetname" "")
@@
     (fp_line (start -2.55 -0.2) (end -1.8 -0.2)
       (stroke (width 0.12) (type solid)) (layer "F.SilkS"))
-    (fp_line (start -1.8 -0.2) (end -1.8 1.14)
+    (fp_line (start -1.8 -0.2) (end -1.8 2.75)
+      (stroke (width 0.12) (type solid)) (layer "F.SilkS"))
+    (fp_line (start -1.8 2.75) (end 5 2.75)
       (stroke (width 0.12) (type solid)) (layer "F.SilkS"))
     (fp_line (start -1.6 -2.75) (end -2.85 -2.75)
@@
     (fp_line (start 0.75 -1.7) (end 9.25 -1.7)
       (stroke (width 0.12) (type solid)) (layer "F.SilkS"))
-    (fp_line (start 5 2.75) (end -0.74 2.75)
-      (stroke (width 0.12) (type solid)) (layer "F.SilkS"))
     (fp_line (start 9.25 -2.45) (end 0.75 -2.45)
       (stroke (width 0.12) (type solid)) (layer "F.SilkS"))
@@
     (fp_line (start 12.45 3.4) (end 12.45 -2.35)
       (stroke (width 0.1) (type solid)) (layer "F.Fab"))
-    (pad "" np_thru_hole circle (at -1.6 2) (size 1.2 1.2) (drill 1.2) (layers "*.Cu" "*.Mask"))
-    (pad "1" thru_hole roundrect (at 0 0) (size 1.7 1.95) (drill 0.95) (layers "*.Cu" "*.Mask") (roundrect_rratio 0.1470588235)
+    (pad "1" thru_hole roundrect (at 0 0) (size 1.7 1.95) (drill 0.95) (layers "*.Cu" "*.Mask") (roundrect_rratio 0.147059)
       (net 16 "Net-(J2-Pin_1)") (pinfunction "Pin_1") (pintype "passive"))
     (pad "2" thru_hole oval (at 2.5 0) (size 1.7 1.95) (drill 0.95) (layers "*.Cu" "*.Mask")
@@
     (pad "5" thru_hole oval (at 10 0) (size 1.7 1.95) (drill 0.95) (layers "*.Cu" "*.Mask")
       (net 20 "Net-(J2-Pin_5)") (pinfunction "Pin_5") (pintype "passive"))
-    (model "${KICAD6_3DMODEL_DIR}/Connector_JST.3dshapes/JST_XH_B5B-XH-AM_1x05_P2.50mm_Vertical.wrl"
+    (model "${KICAD6_3DMODEL_DIR}/Connector_JST.3dshapes/JST_XH_B5B-XH-A_1x05_P2.50mm_Vertical.wrl"
       (offset (xyz 0 0 0))
       (scale (xyz 1 1 1))
